Commit message: 删除X5机器人相关的URDF和STL文件，并更新X5A机器人及其夹爪的相关代码和文档。需要更改对应夹爪与机械臂的资源文件(xml)

File: models/X5A/urdf/X5A.urdf (robot description, URDF)
Before this commit: robot ultron2_urdf_g, 9 links, 8 joints
Links:
- removed link eef_link
- added link link8, mass 0.064798; collision mesh filename=package://X5A/meshes/link8.STL; visual mesh filename=package://X5A/meshes/link8.STL
- link base_link: mass 0.44235 -> 0.43995; geometry collision mesh filename=package://X5A/meshes/base_link.STL; visual mesh filename=package://X5A/meshes/base_link.STL
- link link1: mass 0.085583 -> 0.066982; geometry collision mesh filename=package://X5A/meshes/link1.STL; visual mesh filename=package://X5A/meshes/link1.STL
- link link2: mass 1.02244259916853 -> 1.0795; geometry collision mesh filename=package://X5A/meshes/link2.STL; visual mesh filename=package://X5A/meshes/link2.STL
- link link3: mass 0.84083747270065 -> 0.54534; geometry collision mesh filename=package://X5A/meshes/link3.STL; visual mesh filename=package://X5A/meshes/link3.STL
- link link4: mass 0.43314458599201 -> 0.11714; geometry collision mesh filename=package://X5A/meshes/link4.STL; visual mesh filename=package://X5A/meshes/link4.STL
- link link5: mass 0.552346497691693 -> 0.63488; geometry collision mesh filename=package://X5A/meshes/link5.STL; visual mesh filename=package://X5A/meshes/link5.STL
- link link6: mass 0.369986281234796 -> 0.44089; geometry collision mesh filename=package://X5A/meshes/link6.STL; visual mesh filename=package://X5A/meshes/link6.STL
- link link7: mass 0.66 -> 0.064798; geometry collision mesh filename=package://X5A/meshes/link7.STL; visual mesh filename=package://X5A/meshes/link7.STL
Joints:
- removed joint gripper_fixed_joint
- added joint joint8: type prismatic, parent link6, child link8, origin xyz=0.08657 -0.0249 -0.00024366 rpy=0 0 0, axis 0 -1 0, limit lower=0 upper=0.044 effort=100 velocity=1000
- joint joint1: axis 0 1 0 -> 0 0 1; origin xyz=0 0.0605 0 rpy=0 0 0 -> xyz=0 0 0.0605 rpy=0 0 0
- joint joint2: axis 1 0 0 -> 0 1 0; origin xyz=0.03125 0.059 0 rpy=0 0 3.1416 -> xyz=0.02 0 0.04 rpy=0 0 0
- joint joint3: axis 0 0 1 -> 0 1 0; origin xyz=0.03125 0 -0.0905 rpy=3.1416 0 3.1416 -> xyz=-0.264 0 0 rpy=3.1416 0 0
- joint joint4: origin xyz=0 0.03125 0.2125 rpy=0 0 0 -> xyz=0.245 0 -0.056 rpy=0 0 0
- joint joint5: axis 1 0 0 -> 0 0 1; origin xyz=0.0935 -0.03125 0 rpy=3.1416 0 0 -> xyz=0.06775 0.0005 -0.0865 rpy=0 0 0
- joint joint6: axis 0 1 0 -> 1 0 0; origin xyz=0.1615 -0.03425 0 rpy=-3.1416 0 0 -> xyz=0.02895 0 0.0865 rpy=-3.1416 0 0
- joint joint7: axis 0 0 -1 -> 0 1 0; limit lower=-10 upper=10 effort=100 velocity=1000 -> lower=0 upper=0.044 effort=100 velocity=1000; origin xyz=0 -0.03425 0.022 rpy=-3.1416 0 0 -> xyz=0.08657 0.024896 -0.0002436 rpy=0 0 0; type revolute -> prismatic
